File: macboard.brd (EAGLE design)
At the start: 71.8 x 54.6 mm, 2 parts, among them X1 5566-14

Commit message: audio
Parts:
- added CN1: (no value), adafruit:JST-PH-2-THM
Connections:
- new net AUDIO: CN1.2
- net GND: now also CN1.1
Changed lines of the file:
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@@
 <attribute name="OC_FARNELL" value="unknown" x="46.99" y="54.61" size="1.27" layer="27" display="off"/>
 </element>
+<element name="CN1" library="adafruit" package="JST-PH-2-THM" value="" x="38.1" y="40.64"/>
 </elements>
 <signals>
@@
 <contactref element="X1" pad="5"/>
 <contactref element="X1" pad="8"/>
+<contactref element="CN1" pad="1"/>
+<wire x1="21.59" y1="17.145" x2="39.1" y2="40.64" width="0" layer="19" extent="1-1"/>
 </signal>
 <signal name="VDD_3V3EXP">
@@
 <contactref element="X1" pad="11"/>
 </signal>
+<signal name="AUDIO">
+<contactref element="CN1" pad="2"/>
+</signal>
 </signals>
