File: macboard.sch (EAGLE design)
At the start: 2 parts, among them X1 5566-14

Commit message: audio
Parts:
- added CN1: (no value), adafruit:JST_2PIN-THM
Connections:
- new net AUDIO: CN1.1
- net GND: now also CN1.2
Changed lines of the file:
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@@
 <part name="U$1" library="adafruit" deviceset="BEAGLEBONE_OUTLINE" device=""/>
 <part name="X1" library="con-molex" deviceset="5566-14" device=""/>
+<part name="CN1" library="adafruit" deviceset="JST_2PIN" device="-THM"/>
 </parts>
 <sheets>
@@
 <instance part="X1" gate="-13" x="142.24" y="93.98"/>
 <instance part="X1" gate="-14" x="142.24" y="91.44"/>
+<instance part="CN1" gate="G$1" x="144.78" y="73.66"/>
 </instances>
 <busses>
@@
 <label x="127" y="106.68" size="1.778" layer="95"/>
 </segment>
+<segment>
+<pinref part="CN1" gate="G$1" pin="2"/>
+<wire x1="142.24" y1="73.66" x2="127" y2="73.66" width="0.1524" layer="91"/>
+<label x="127" y="73.66" size="1.778" layer="95"/>
+</segment>
 </net>
 <net name="A_RAW" class="0">
@@
 </segment>
 </net>
+<net name="AUDIO" class="0">
+<segment>
+<pinref part="CN1" gate="G$1" pin="1"/>
+<wire x1="142.24" y1="76.2" x2="127" y2="76.2" width="0.1524" layer="91"/>
+<label x="127" y="78.74" size="1.778" layer="95"/>
+</segment>
+</net>
